Commit message: Update documentation and joint rotations

File: Martha_ws/src/martha_description/urdf/martha_joints.xacro (robot description, xacro)
@@ -164,5 +164,5 @@
   <parent link="r_waist_1"/>
   <child link="r_thigh_1"/>
-  <axis xyz="1.0 0.0 0.0"/>
+  <axis xyz="-1.0 0.0 0.0"/>
   <limit lower="-3.14159" upper="3.14159" effort="1000.0" velocity="0.01"/>
   <physics>
@@ -177,5 +177,5 @@
   <parent link="l_waist_1"/>
   <child link="l_thigh_1"/>
-  <axis xyz="1.0 0.0 0.0"/>
+  <axis xyz="-1.0 0.0 0.0"/>
   <limit lower="-3.14159" upper="3.14159" effort="1000.0" velocity="0.01"/>
   <physics>
@@ -190,5 +190,5 @@
   <parent link="l_thigh_1"/>
   <child link="l_shin_1"/>
-  <axis xyz="-1.0 -0.0 -0.0"/>
+  <axis xyz="1.0 -0.0 -0.0"/>
   <limit lower="-3.14159" upper="3.14159" effort="1000.0" velocity="0.01"/>
   <physics>
@@ -203,5 +203,5 @@
   <parent link="r_thigh_1"/>
   <child link="r_shin_1"/>
-  <axis xyz="-1.0 -0.0 -0.0"/>
+  <axis xyz="1.0 -0.0 -0.0"/>
   <limit lower="-3.14159" upper="3.14159" effort="1000.0" velocity="0.01"/>
   <physics>
@@ -216,5 +216,5 @@
   <parent link="r_shin_1"/>
   <child link="r_ankle_1"/>
-  <axis xyz="1.0 0.0 0.0"/>
+  <axis xyz="-1.0 0.0 0.0"/>
   <limit lower="-3.14159" upper="3.14159" effort="1000.0" velocity="0.01"/>
   <physics>
@@ -229,5 +229,5 @@
   <parent link="l_shin_1"/>
   <child link="l_ankle_1"/>
-  <axis xyz="1.0 0.0 -0.0"/>
+  <axis xyz="-1.0 0.0 -0.0"/>
   <limit lower="-3.14159" upper="3.14159" effort="1000.0" velocity="0.01"/>
   <physics>

Commit message: atualizacao de direcoes das juntas (que deveria ter subido ontem)

File: Martha_ws/src/martha_description/urdf/martha_joints.xacro (robot description, xacro)
@@ -21,5 +21,5 @@
   <parent link="base_link"/>
   <child link="l_shoulder_1"/>
-  <axis xyz="1.0 -0.0 0.0"/>
+  <axis xyz="-1.0 -0.0 0.0"/>
   <limit lower="-3.14159" upper="3.14159" effort="1000.0" velocity="0.01"/>
   <physics>
@@ -60,5 +60,5 @@
   <parent link="base_link"/>
   <child link="neck_1"/>
-  <axis xyz="0.0 0.0 1.0"/>
+  <axis xyz="0.0 0.0 -1.0"/>
   <limit lower="-3.14159" upper="3.14159" effort="1000.0" velocity="0.01"/>
   <physics>
@@ -125,5 +125,5 @@
   <parent link="base_link"/>
   <child link="r_hip_1"/>
-  <axis xyz="-0.0 -0.0 -1.0"/>
+  <axis xyz="-0.0 -0.0 1.0"/>
   <limit lower="-3.14159" upper="3.14159" effort="1000.0" velocity="0.01"/>
   <physics>
@@ -164,5 +164,5 @@
   <parent link="r_waist_1"/>
   <child link="r_thigh_1"/>
-  <axis xyz="-1.0 0.0 0.0"/>
+  <axis xyz="1.0 0.0 0.0"/>
   <limit lower="-3.14159" upper="3.14159" effort="1000.0" velocity="0.01"/>
   <physics>
@@ -177,5 +177,5 @@
   <parent link="l_waist_1"/>
   <child link="l_thigh_1"/>
-  <axis xyz="-1.0 0.0 0.0"/>
+  <axis xyz="1.0 0.0 0.0"/>
   <limit lower="-3.14159" upper="3.14159" effort="1000.0" velocity="0.01"/>
   <physics>
@@ -216,5 +216,5 @@
   <parent link="r_shin_1"/>
   <child link="r_ankle_1"/>
-  <axis xyz="-1.0 0.0 0.0"/>
+  <axis xyz="1.0 0.0 0.0"/>
   <limit lower="-3.14159" upper="3.14159" effort="1000.0" velocity="0.01"/>
   <physics>
@@ -229,5 +229,5 @@
   <parent link="l_shin_1"/>
   <child link="l_ankle_1"/>
-  <axis xyz="-1.0 0.0 -0.0"/>
+  <axis xyz="1.0 0.0 -0.0"/>
   <limit lower="-3.14159" upper="3.14159" effort="1000.0" velocity="0.01"/>
   <physics>
