Commit message: Update marta_joints.xacro
Corrigido ângulos

File: Marta_ws/src/marta_description/urdf/marta_joints.xacro (robot description, xacro)
@@ -8,5 +8,5 @@
   <parent link="base_link"/>
   <child link="neck_1"/>
-  <axis xyz="-0.0 0.0 1.0"/>
+  <axis xyz="-0.0 0.0 -1.0"/>
   <!-- <dynamics damping="0.1" /> -->
   <limit lower="-3.14159" upper="3.14159" effort="1000.0" velocity="0.01"/>
@@ -16,5 +16,5 @@
   <parent link="neck_1"/>
   <child link="head_1"/>
-  <axis xyz="-0.0 1.0 -0.0"/>
+  <axis xyz="-0.0 -1.0 -0.0"/>
   <!-- <dynamics damping="0.1" /> -->
   <limit lower="-3.14159" upper="3.14159" effort="1000.0" velocity="0.01"/>
@@ -56,5 +56,5 @@
   <parent link="r_waist_1"/>
   <child link="r_thigh_1"/>
-  <axis xyz="0.0 -1.0 -0.0"/>
+  <axis xyz="0.0 1.0 -0.0"/>
   <!-- <dynamics damping="0.1" /> -->
   <limit lower="-3.14159" upper="3.14159" effort="1000.0" velocity="0.01"/>
@@ -72,5 +72,5 @@
   <parent link="r_thigh_1"/>
   <child link="r_shin_1"/>
-  <axis xyz="-0.0 -1.0 -0.0"/>
+  <axis xyz="-0.0 1.0 -0.0"/>
   <!-- <dynamics damping="0.1" /> -->
   <limit lower="-3.14159" upper="3.14159" effort="1000.0" velocity="0.01"/>
@@ -88,5 +88,5 @@
   <parent link="l_shin_1"/>
   <child link="l_ankle_1"/>
-  <axis xyz="-0.0 -1.0 -0.0"/>
+  <axis xyz="-0.0 1.0 -0.0"/>
   <!-- <dynamics damping="0.1" /> -->
   <limit lower="-3.14159" upper="3.14159" effort="1000.0" velocity="0.01"/>
@@ -112,5 +112,5 @@
   <parent link="base_link"/>
   <child link="l_shoulder_1"/>
-  <axis xyz="0.0 1.0 0.0"/>
+  <axis xyz="0.0 -1.0 0.0"/>
   <!-- <dynamics damping="0.1" /> -->
   <limit lower="-3.14159" upper="3.14159" effort="1000.0" velocity="0.01"/>
@@ -136,5 +136,5 @@
   <parent link="r_shoulder_1"/>
   <child link="r_arm_1"/>
-  <axis xyz="1.0 0.0 -0.0"/>
+  <axis xyz="-1.0 0.0 -0.0"/>
   <!-- <dynamics damping="0.1" /> -->
   <limit lower="-3.14159" upper="3.14159" effort="1000.0" velocity="0.01"/>
@@ -160,5 +160,5 @@
   <parent link="l_arm_1"/>
   <child link="l_hand_1"/>
-  <axis xyz="-0.0 1.0 0.0"/>
+  <axis xyz="-0.0 -1.0 0.0"/>
   <!-- <dynamics damping="0.1" /> -->
   <limit lower="-3.14159" upper="3.14159" effort="1000.0" velocity="0.01"/>
